File: Reader.kicad_sch (KiCad schematic)
At the start: 42 parts, among them J1 Conn_01x04, J2 Amphenol Dubox ‎76383-402LF‎, J3 Conn_01x04, J4 Conn_01x08, J5 Conn_01x10, J6 Conn_01x03, J7 Conn_01x02, Q1 2N7002, Q2 2N7002, Q3 2N7002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

Commit message: Add changelog file
Other:
- note removed: "TODO: - Resistor values on silk? Done: - Removed optional from pulldowns, made value 1k - Added series resistors for button input - Added C2 to suppress output pin pulses - Enlarged mounting holes from 2.5mm to 3.2mm - Marked LED polarity on silkscreen - Reduced overly wide thermal reliefs due to wide GND traces - Added C3 as input supply buffer cap - Change to hand soldering footprints for trans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"
Changed lines of the file:
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@@
-		)
-	)
-	(text "TODO:\n - Resistor values on silk?\n\nDone:\n - Removed optional from pulldowns, made value 1k\n - Added series resistors for button input\n - Added C2 to suppress output pin pulses\n - Enlarged mounting holes from 2.5mm to 3.2mm\n - Marked LED polarity on silkscreen\n - Reduced overly wide thermal reliefs due to wide GND traces\n - Added C3 as input supply buffer cap\n - Change to hand soldering footprints for transistors"
-		(exclude_from_sim no)
-		(at 116.84 152.4 0)
-		(effects
-			(font
-				(size 1.27 1.27)
-			)
-			(justify left bottom)
 		)
 	)
