File: PCB/Reader.kicad_pcb (KiCad board)
At the start: 2 copper layers, 40.4 x 60 mm, 43 parts, among them J1 Conn_01x04, J2 Amphenol Dubox ‎76383-402LF‎, J3 Conn_01x04, J4 Conn_01x08, J5 Conn_01x10, J6 Conn_01x03, J7 Conn_01x02, Q1 2N7002, Q2 2N7002, Q3 2N7002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

Commit message: Use CERN-OHL-P v2+ license
Other:
- board text added: "CERN-OHL-P v2+"
- board text removed: "CC-BY 4.0"
Changed lines of the file:
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@@
 	)
 	(paper "A4")
+	(title_block
+		(title "Doorlockd Reader PCB")
+		(comment 1 "Copyright 2021-2025 Matthijs Kooijman <matthijs@stdin.nl>\n")
+		(comment 2 "Licensed under CERN-OHL-P v2 or any later version")
+	)
 	(layers
 		(0 "F.Cu" signal)
@@
 		)
 	)
-	(gr_text "CC-BY 4.0"
+	(gr_text "CERN-OHL-P v2+"
 		(at 112 82 0)
 		(layer "B.SilkS")
